File: RP2350Adev/RP2350Adev.kicad_sch (KiCad schematic)
At the start: 39 parts, among them J401 UART, J402 DEBUG, U401 MCP1702T-3302E_CB, U402 W25Q32JV, U403 RP2350A, X401 IQXO-791

Commit message: fix footprint errors
Parts:
- U401: value MCP1702T-3302E_CB -> LD1117S33TR_SOT223; footprint Package_TO_SOT_SMD:SOT-23 -> Package_TO_SOT_SMD:SOT-223-3_TabPin2; symbol Eclectronics:MCP1702T-3302E_CB -> Regulator_Linear:LD1117S33TR_SOT223
Changed lines of the file:
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@@
 	(wire
 		(pts
-			(xy 29.21 130.81) (xy 31.75 130.81)
+			(xy 29.21 130.81) (xy 36.83 130.81)
 		)
 		(stroke
@@
 	(wire
 		(pts
-			(xy 57.15 130.81) (xy 59.69 130.81)
-		)
-		(stroke
-			(width 0)
-			(type default)
-		)
-	)
-	(wire
-		(pts
 			(xy 111.76 124.46) (xy 113.03 124.46)
 		)
@@
 	(wire
 		(pts
+			(xy 44.45 138.43) (xy 44.45 143.51)
+		)
+		(stroke
+			(width 0)
+			(type default)
+		)
+	)
+	(wire
+		(pts
 			(xy 111.76 139.7) (xy 111.76 144.78)
 		)
@@
 	(wire
 		(pts
+			(xy 52.07 130.81) (xy 59.69 130.81)
+		)
+		(stroke
+			(width 0)
+			(type default)
+		)
+	)
+	(wire
+		(pts
 			(xy 58.42 68.58) (xy 59.69 68.58)
 		)
@@
 				)
 			)
+			(project "RP2350Adev"
+				(path "/4930e8a3-0a58-4861-9c4c-0d8b2139987a"
+					(reference "J?")
+					(unit 1)
+				)
+			)
 		)
 	)
@@
 				)
 			)
+			(project "RP2350Adev"
+				(path "/4930e8a3-0a58-4861-9c4c-0d8b2139987a"
+					(reference "#PWR?")
+					(unit 1)
+				)
+			)
 		)
 	)
@@
 	)
 	(symbol
-		(lib_id "Eclectronics:MCP1702T-3302E_CB")
-		(at 44.45 133.35 0)
+		(lib_id "Regulator_Linear:LD1117S33TR_SOT223")
+		(at 44.45 130.81 0)
 		(unit 1)
 		(exclude_from_sim no)
@@
 		(dnp no)
 		(property "Reference" "U401"
-			(at 36.83 123.19 0)
+			(at 36.83 120.65 0)
 			(effects
 				(font
@@
 			)
 		)
-		(property "Value" "MCP1702T-3302E_CB"
-			(at 36.83 125.73 0)
+		(property "Value" "LD1117S33TR_SOT223"
+			(at 44.45 127.635 0)
 			(effects
 				(font
@@
 			)
 		)
-		(property "Footprint" "Package_TO_SOT_SMD:SOT-23"
-			(at 44.45 132.08 0)
+		(property "Footprint" "Package_TO_SOT_SMD:SOT-223-3_TabPin2"
+			(at 44.45 125.73 0)
 			(effects
 				(font
-					(size 1.524 1.524)
+					(size 1.27 1.27)
 				)
 				(hide yes)
 			)
 		)
-		(property "Datasheet" ""
-			(at 44.45 132.08 0)
+		(property "Datasheet" "http://www.st.com/st-web-ui/static/active/en/resource/technical/document/datasheet/CD00000544.pdf"
+			(at 46.99 137.16 0)
 			(effects
 				(font
-					(size 1.524 1.524)
+					(size 1.27 1.27)
 				)
 				(hide yes)
 			)
 		)
-		(property "Description" ""
-			(at 44.45 133.35 0)
+		(property "Description" "800mA Fixed Low Drop Positive Voltage Regulator, Fixed Output 3.3V, SOT-223"
+			(at 44.45 130.81 0)
 			(effects
 				(font
 					(size 1.27 1.27)
 				)
+				(hide yes)
 			)
 		)
@@
 		)
 	)
+	(sheet_instances
+		(path "/"
+			(page "1")
+		)
+	)
+	(embedded_fonts no)
 )
