File: RP2350Adev/USB_Mux_Periph.kicad_sch (KiCad schematic)
At the start: 3 parts, among them J5 USB_A_Male, J6 USB_A_Female, U5 TS3USB30EDGSR

Commit message: Muxful Developings
Parts:
- added SW1: SW_DIP_x06, symbol Switch:SW_DIP_x06
- added U1: TS3USB3031RMGR, RMG12_TEX, symbol Eclectronics:TS3USB3031RMGR
- renumbered J5 to J1, J6 to J2, U5 to U2
Connections:
- net +5V: now also U1.12 (VCC); no longer J1.1 (VBUS)
- net GND: now also U1.9 (GND)
- net at U2.4 (D+): now also U1.11 (D+)
- net at U2.6 (D-): now also U1.10 (D-)

Commit message: Muxful Schematics Done (Added external standalone 5V supply USB-C connector)
Parts:
- added J3: USB4105-GF-A, Eclectronics:USB4105-GF-A, symbol Eclectronics:USB4105-GF-A
- added R1, R2, R3, R4: 10K, symbol Device:R
- added R5, R6: 5.1K, Resistor_SMD:R_0402_1005Metric, symbol Device:R
- renumbered U1 to M1, U2 to M2
Connections:
- net +5V: now also J1.1 (VBUS), J3.A4B9 (VBUS), J3.B4A9 (VBUS); no longer M1.12 (VCC), M2.10 (VCC)
- net GND: now also J3.A1B12 (GND), J3.B1A12 (GND), J3.S1 (SHELL), J3.S2 (SHELL), J3.S3 (SHELL), J3.S4 (SHELL), R1.2, R2.2, R3.2, R4.2, R5.2, R6.2
- net MUX1_S0: now reaches M1.1 (SEL0)
- net MUX1_S0: now also SW1.1, R1.1
- net MUX1_S1: now reaches M1.2 (SEL1)
- net MUX1_S1: now also SW1.2, R2.1
- net D1+: now reaches M1.3 (USB1+)
- net D1-: now reaches M1.4 (USB1-)
- net D2+: now reaches M1.5 (USB2+)
- net D2-: now reaches M1.6 (USB2-)
- net D3+: now reaches M1.7 (MHL+)
- net D3-: now reaches M1.8 (MHL-)
- net MUX2_S: now reaches M2.1 (S)
- net MUX2_S: now also SW1.4, R4.1
- net MUX2_OE: now reaches M2.9 (~{OE})
- net MUX2_OE: now also SW1.3, R3.1
- net +3V3: now reaches SW1.10
- net +3V3: now also M1.12 (VCC), M2.10 (VCC), SW1.11, SW1.12, SW1.9
- new net: J3.B5 (CC2), R5.1
- new net: J3.A5 (CC1), R6.1
- new net: J3.A6 (D+), J3.B6 (D+)
- new net: J3.A7 (D-), J3.B7 (D-)
- no-connect marks 0 -> 8
Other:
- moved on the sheet: SW1

Commit message: Muxful Assignings of Components and Foots
Parts:
- J1: footprint Connector_USB:USB_A_Connfly_DS1098_Horizontal -> Eclectronics:USB_A_0480370001
- J2: footprint (none) -> Connector_USB:USB_A_Stewart_SS-52100-001_Horizontal
- M1: footprint RMG12_TEX -> Eclectronics:RMG12_TEX
- R1, R2, R3, R4: footprint (none) -> Capacitor_SMD:C_0402_1005Metric
- R5, R6: footprint Resistor_SMD:R_0402_1005Metric -> Capacitor_SMD:C_0402_1005Metric
- SW1: footprint (none) -> Button_Switch_THT:SW_DIP_SPSTx06_Piano_10.8x16.8mm_W7.62mm_P2.54mm
Changed lines of the file:
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@@
 		(dnp no)
 		(fields_autoplaced yes)
-		(property "Reference" "#PWR?"
+		(property "Reference" "#PWR0105"
 			(at 95.25 87.63 0)
 			(effects
@@
 			(project "USB_Mux_Periph"
 				(path "/1a5d876a-e386-4d19-8f87-fb5cfd2ba4be"
-					(reference "#PWR?")
+					(reference "#PWR0105")
 					(unit 1)
 				)
@@
 			)
 		)
-		(property "Footprint" ""
+		(property "Footprint" "Connector_USB:USB_A_Stewart_SS-52100-001_Horizontal"
 			(at 53.34 80.01 0)
 			(effects
@@
 			)
 		)
-		(property "Footprint" "Resistor_SMD:R_0402_1005Metric"
+		(property "Footprint" "Capacitor_SMD:C_0402_1005Metric"
 			(at 252.222 55.88 90)
 			(effects
@@
 			)
 		)
-		(property "Footprint" "Connector_USB:USB_A_Connfly_DS1098_Horizontal"
+		(property "Footprint" "Eclectronics:USB_A_0480370001"
 			(at 53.34 46.99 0)
 			(effects
@@
 			)
 		)
-		(property "Footprint" ""
+		(property "Footprint" "Capacitor_SMD:C_0402_1005Metric"
 			(at 42.672 109.22 90)
 			(effects
@@
 			)
 		)
-		(property "Footprint" "RMG12_TEX"
+		(property "Footprint" "Eclectronics:RMG12_TEX"
 			(at 190.5 62.23 0)
 			(effects
@@
 			)
 		)
-		(property "Footprint" ""
+		(property "Footprint" "Capacitor_SMD:C_0402_1005Metric"
 			(at 61.722 111.76 90)
 			(effects
@@
 			)
 		)
-		(property "Footprint" "Resistor_SMD:R_0402_1005Metric"
+		(property "Footprint" "Capacitor_SMD:C_0402_1005Metric"
 			(at 261.112 55.88 90)
 			(effects
@@
 			)
 		)
-		(property "Footprint" ""
+		(property "Footprint" "Capacitor_SMD:C_0402_1005Metric"
 			(at 80.772 114.3 90)
 			(effects
@@
 			)
 		)
-		(property "Footprint" ""
+		(property "Footprint" "Capacitor_SMD:C_0402_1005Metric"
 			(at 98.552 116.84 90)
 			(effects
@@
 		(dnp no)
 		(fields_autoplaced yes)
-		(property "Reference" "#PWR?"
+		(property "Reference" "#PWR0103"
 			(at 46.99 63.5 0)
 			(effects
@@
 			(project "USB_Mux_Periph"
 				(path "/1a5d876a-e386-4d19-8f87-fb5cfd2ba4be"
-					(reference "#PWR?")
+					(reference "#PWR0103")
 					(unit 1)
 				)
@@
 		(dnp no)
 		(fields_autoplaced yes)
-		(property "Reference" "#PWR?"
+		(property "Reference" "#PWR0104"
 			(at 59.69 73.66 0)
 			(effects
@@
 			(project "USB_Mux_Periph"
 				(path "/1a5d876a-e386-4d19-8f87-fb5cfd2ba4be"
-					(reference "#PWR?")
+					(reference "#PWR0104")
 					(unit 1)
 				)
@@
 		(dnp no)
 		(fields_autoplaced yes)
-		(property "Reference" "#PWR?"
+		(property "Reference" "#PWR0102"
 			(at 46.99 96.52 0)
 			(effects
@@
 			(project "USB_Mux_Periph"
 				(path "/1a5d876a-e386-4d19-8f87-fb5cfd2ba4be"
-					(reference "#PWR?")
+					(reference "#PWR0102")
 					(unit 1)
 				)
@@
 		(dnp no)
 		(fields_autoplaced yes)
-		(property "Reference" "#PWR06"
+		(property "Reference" "#PWR0101"
 			(at 226.06 78.74 0)
 			(effects
@@
 			(project "USB_Mux_Periph"
 				(path "/1a5d876a-e386-4d19-8f87-fb5cfd2ba4be"
-					(reference "#PWR06")
+					(reference "#PWR0101")
 					(unit 1)
 				)
@@
 			)
 		)
-		(property "Footprint" ""
+		(property "Footprint" "Button_Switch_THT:SW_DIP_SPSTx06_Piano_10.8x16.8mm_W7.62mm_P2.54mm"
 			(at 115.57 113.03 0)
 			(effects

Commit message: Combine subsheets
Parts:
- renumbered J1 to J7, J2 to J8, J3 to J9, R1 to R18, R2 to R19, R3 to R20, R4 to R21, R5 to R22, R6 to R23, M2 to U8
Changed lines of the file:
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@@
 		(dnp no)
 		(fields_autoplaced yes)
-		(property "Reference" "#PWR0105"
+		(property "Reference" "#PWR075"
 			(at 95.25 87.63 0)
 			(effects
@@
 			(project "RP2350Adev"
 				(path "/1f57b86c-11e7-4ea8-8f36-592c0861a25b/035fadad-9eba-4726-a427-88058f0933c7"
-					(reference "#PWR07")
+					(reference "#PWR075")
 					(unit 1)
 				)
@@
 		(dnp no)
 		(fields_autoplaced yes)
-		(property "Reference" "#PWR01"
+		(property "Reference" "#PWR078"
 			(at 147.32 66.04 0)
 			(effects
@@
 				)
 			)
+			(project "main"
+				(path "/1f57b86c-11e7-4ea8-8f36-592c0861a25b/035fadad-9eba-4726-a427-88058f0933c7"
+					(reference "#PWR078")
+					(unit 1)
+				)
+			)
 		)
 	)
@@
 		(dnp no)
 		(fields_autoplaced yes)
-		(property "Reference" "J2"
+		(property "Reference" "J8"
 			(at 49.53 66.04 0)
 			(effects
@@
 			(project ""
 				(path "/1f57b86c-11e7-4ea8-8f36-592c0861a25b/035fadad-9eba-4726-a427-88058f0933c7"
-					(reference "J6")
+					(reference "J8")
 					(unit 1)
 				)
@@
 		(dnp no)
 		(fields_autoplaced yes)
-		(property "Reference" "R5"
+		(property "Reference" "R22"
 			(at 256.54 54.6099 0)
 			(effects
@@
 				)
 			)
+			(project "main"
+				(path "/1f57b86c-11e7-4ea8-8f36-592c0861a25b/035fadad-9eba-4726-a427-88058f0933c7"
+					(reference "R22")
+					(unit 1)
+				)
+			)
 		)
 	)
@@
 		(dnp no)
 		(fields_autoplaced yes)
-		(property "Reference" "#PWR08"
+		(property "Reference" "#PWR082"
 			(at 254 66.04 0)
 			(effects
@@
 				)
 			)
+			(project "main"
+				(path "/1f57b86c-11e7-4ea8-8f36-592c0861a25b/035fadad-9eba-4726-a427-88058f0933c7"
+					(reference "#PWR082")
+					(unit 1)
+				)
+			)
 		)
 	)
@@
 		(dnp no)
 		(fields_autoplaced yes)
-		(property "Reference" "J1"
+		(property "Reference" "J7"
 			(at 49.53 33.02 0)
 			(effects
@@
 			(project ""
 				(path "/1f57b86c-11e7-4ea8-8f36-592c0861a25b/035fadad-9eba-4726-a427-88058f0933c7"
-					(reference "J5")
+					(reference "J7")
 					(unit 1)
 				)
@@
 		(dnp no)
 		(fields_autoplaced yes)
-		(property "Reference" "R1"
+		(property "Reference" "R18"
 			(at 46.99 107.9499 0)
 			(effects
@@
 				)
 			)
+			(project "main"
+				(path "/1f57b86c-11e7-4ea8-8f36-592c0861a25b/035fadad-9eba-4726-a427-88058f0933c7"
+					(reference "R18")
+					(unit 1)
+				)
+			)
 		)
 	)
@@
 		(dnp no)
 		(fields_autoplaced yes)
-		(property "Reference" "#PWR02"
+		(property "Reference" "#PWR077"
 			(at 142.24 85.09 0)
 			(effects
@@
 				)
 			)
+			(project "main"
+				(path "/1f57b86c-11e7-4ea8-8f36-592c0861a25b/035fadad-9eba-4726-a427-88058f0933c7"
+					(reference "#PWR077")
+					(unit 1)
+				)
+			)
 		)
 	)
@@
 		(on_board yes)
 		(dnp no)
-		(property "Reference" "#PWR07"
+		(property "Reference" "#PWR081"
 			(at 248.92 68.58 0)
 			(effects
@@
 				)
 			)
+			(project "main"
+				(path "/1f57b86c-11e7-4ea8-8f36-592c0861a25b/035fadad-9eba-4726-a427-88058f0933c7"
+					(reference "#PWR081")
+					(unit 1)
+				)
+			)
 		)
 	)
@@
 		(dnp no)
 		(fields_autoplaced yes)
-		(property "Reference" "#PWR03"
+		(property "Reference" "#PWR069"
 			(at 44.45 130.81 0)
 			(effects
@@
 				(path "/1a5d876a-e386-4d19-8f87-fb5cfd2ba4be"
 					(reference "#PWR03")
+					(unit 1)
+				)
+			)
+			(project "main"
+				(path "/1f57b86c-11e7-4ea8-8f36-592c0861a25b/035fadad-9eba-4726-a427-88058f0933c7"
+					(reference "#PWR069")
 					(unit 1)
 				)
@@
 				)
 			)
+			(project "main"
+				(path "/1f57b86c-11e7-4ea8-8f36-592c0861a25b/035fadad-9eba-4726-a427-88058f0933c7"
+					(reference "M1")
+					(unit 1)
+				)
+			)
 		)
 	)
@@
 		(dnp no)
 		(fields_autoplaced yes)
-		(property "Reference" "R2"
+		(property "Reference" "R19"
 			(at 66.04 110.4899 0)
 			(effects
@@
 				(path "/1a5d876a-e386-4d19-8f87-fb5cfd2ba4be"
 					(reference "R2")
+					(unit 1)
+				)
+			)
+			(project "main"
+				(path "/1f57b86c-11e7-4ea8-8f36-592c0861a25b/035fadad-9eba-4726-a427-88058f0933c7"
+					(reference "R19")
 					(unit 1)
 				)
@@
 		(on_board yes)
 		(dnp no)
-		(property "Reference" "M2"
+		(property "Reference" "U8"
 			(at 93.1067 57.15 0)
 			(effects
@@
 			(project "RP2350Adev"
 				(path "/1f57b86c-11e7-4ea8-8f36-592c0861a25b/035fadad-9eba-4726-a427-88058f0933c7"
-					(reference "U5")
+					(reference "U8")
 					(unit 1)
 				)
@@
 		(dnp no)
 		(fields_autoplaced yes)
-		(property "Reference" "R6"
+		(property "Reference" "R23"
 			(at 265.43 54.6099 0)
 			(effects
@@
 				)
 			)
+			(project "main"
+				(path "/1f57b86c-11e7-4ea8-8f36-592c0861a25b/035fadad-9eba-4726-a427-88058f0933c7"
+					(reference "R23")
+					(unit 1)
+				)
+			)
 		)
 	)
@@
 		(dnp no)
 		(fields_autoplaced yes)
-		(property "Reference" "#PWR04"
+		(property "Reference" "#PWR076"
 			(at 129.54 109.22 0)
 			(effects
@@
 				)
 			)
+			(project "main"
+				(path "/1f57b86c-11e7-4ea8-8f36-592c0861a25b/035fadad-9eba-4726-a427-88058f0933c7"
+					(reference "#PWR076")
+					(unit 1)
+				)
+			)
 		)
 	)
@@
 		(dnp no)
 		(fields_autoplaced yes)
-		(property "Reference" "#PWR09"
+		(property "Reference" "#PWR074"
 			(at 95.25 60.96 0)
 			(effects
@@
 				)
 			)
+			(project "main"
+				(path "/1f57b86c-11e7-4ea8-8f36-592c0861a25b/035fadad-9eba-4726-a427-88058f0933c7"
+					(reference "#PWR074")
+					(unit 1)
+				)
+			)
 		)
 	)
@@
 		(dnp no)
 		(fields_autoplaced yes)
-		(property "Reference" "#PWR06"
+		(property "Reference" "#PWR080"
 			(at 248.92 35.56 0)
 			(effects
@@
 				)
 			)
+			(project "main"
+				(path "/1f57b86c-11e7-4ea8-8f36-592c0861a25b/035fadad-9eba-4726-a427-88058f0933c7"
+					(reference "#PWR080")
+					(unit 1)
+				)
+			)
 		)
 	)
@@
 		(dnp no)
 		(fields_autoplaced yes)
-		(property "Reference" "#PWR012"
+		(property "Reference" "#PWR083"
 			(at 262.89 66.04 0)
 			(effects
@@
 				)
 			)
+			(project "main"
+				(path "/1f57b86c-11e7-4ea8-8f36-592c0861a25b/035fadad-9eba-4726-a427-88058f0933c7"
+					(reference "#PWR083")
+					(unit 1)
+				)
+			)
 		)
 	)
@@
 		(dnp no)
 		(fields_autoplaced yes)
-		(property "Reference" "R3"
+		(property "Reference" "R20"
 			(at 85.09 113.0299 0)
 			(effects
@@
 				)
 			)
+			(project "main"
+				(path "/1f57b86c-11e7-4ea8-8f36-592c0861a25b/035fadad-9eba-4726-a427-88058f0933c7"
+					(reference "R20")
+					(unit 1)
+				)
+			)
 		)
 	)
@@
 		(dnp no)
 		(fields_autoplaced yes)
-		(property "Reference" "R4"
+		(property "Reference" "R21"
 			(at 102.87 115.5699 0)
 			(effects
@@
 				)
 			)
+			(project "main"
+				(path "/1f57b86c-11e7-4ea8-8f36-592c0861a25b/035fadad-9eba-4726-a427-88058f0933c7"
+					(reference "R21")
+					(unit 1)
+				)
+			)
 		)
 	)
@@
 		(dnp no)
 		(fields_autoplaced yes)
-		(property "Reference" "#PWR0103"
+		(property "Reference" "#PWR070"
 			(at 46.99 63.5 0)
 			(effects
@@
 			(project "RP2350Adev"
 				(path "/1f57b86c-11e7-4ea8-8f36-592c0861a25b/035fadad-9eba-4726-a427-88058f0933c7"
-					(reference "#PWR062")
+					(reference "#PWR070")
 					(unit 1)
 				)
@@
 		(on_board yes)
 		(dnp no)
-		(property "Reference" "J3"
+		(property "Reference" "J9"
 			(at 223.52 25.4 0)
 			(effects
@@
 				)
 			)
+			(project "main"
+				(path "/1f57b86c-11e7-4ea8-8f36-592c0861a25b/035fadad-9eba-4726-a427-88058f0933c7"
+					(reference "J9")
+					(unit 1)
+				)
+			)
 		)
 	)
@@
 		(dnp no)
 		(fields_autoplaced yes)
-		(property "Reference" "#PWR0104"
+		(property "Reference" "#PWR073"
 			(at 59.69 73.66 0)
 			(effects
@@
 			(project "RP2350Adev"
 				(path "/1f57b86c-11e7-4ea8-8f36-592c0861a25b/035fadad-9eba-4726-a427-88058f0933c7"
-					(reference "#PWR061")
+					(reference "#PWR073")
 					(unit 1)
 				)
@@
 		(dnp no)
 		(fields_autoplaced yes)
-		(property "Reference" "#PWR0102"
+		(property "Reference" "#PWR071"
 			(at 46.99 96.52 0)
 			(effects
@@
 			(project "RP2350Adev"
 				(path "/1f57b86c-11e7-4ea8-8f36-592c0861a25b/035fadad-9eba-4726-a427-88058f0933c7"
-					(reference "#PWR063")
+					(reference "#PWR071")
 					(unit 1)
 				)
@@
 		(dnp no)
 		(fields_autoplaced yes)
-		(property "Reference" "#PWR05"
+		(property "Reference" "#PWR072"
 			(at 59.69 40.64 0)
 			(effects
@@
 				)
 			)
+			(project "main"
+				(path "/1f57b86c-11e7-4ea8-8f36-592c0861a25b/035fadad-9eba-4726-a427-88058f0933c7"
+					(reference "#PWR072")
+					(unit 1)
+				)
+			)
 		)
 	)
@@
 		(dnp no)
 		(fields_autoplaced yes)
-		(property "Reference" "#PWR0101"
+		(property "Reference" "#PWR079"
 			(at 226.06 78.74 0)
 			(effects
@@
 				)
 			)
+			(project "main"
+				(path "/1f57b86c-11e7-4ea8-8f36-592c0861a25b/035fadad-9eba-4726-a427-88058f0933c7"
+					(reference "#PWR079")
+					(unit 1)
+				)
+			)
 		)
 	)
@@
 					(reference "SW1")
 					(unit 1)
+				)
+			)
+			(project "main"
+				(path "/1f57b86c-11e7-4ea8-8f36-592c0861a25b/035fadad-9eba-4726-a427-88058f0933c7"
+					(reference "SW1")
+					(unit 1)

Commit message: Layout Assembly Attempt (Components not being transferred as expected, major issues)
Connections:
- net +3V3: now also SW1.1, SW1.2, SW1.3, SW1.4; no longer SW1.10, SW1.11, SW1.12, SW1.9
- net MUX1_S0: now also SW1.12; no longer SW1.1
- net MUX1_S1: now also SW1.11; no longer SW1.2
- net MUX2_OE: now also SW1.10; no longer SW1.3
- net MUX2_S: now also SW1.9; no longer SW1.4
Changed lines of the file:
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@@
 		(dnp no)
 		(fields_autoplaced yes)
-		(property "Reference" "#PWR075"
+		(property "Reference" "#PWR085"
 			(at 95.25 87.63 0)
 			(effects
@@
 			(project "RP2350Adev"
 				(path "/1f57b86c-11e7-4ea8-8f36-592c0861a25b/035fadad-9eba-4726-a427-88058f0933c7"
-					(reference "#PWR075")
+					(reference "#PWR085")
 					(unit 1)
 				)
@@
 		(dnp no)
 		(fields_autoplaced yes)
-		(property "Reference" "#PWR078"
+		(property "Reference" "#PWR088"
 			(at 147.32 66.04 0)
 			(effects
@@
 			(project "main"
 				(path "/1f57b86c-11e7-4ea8-8f36-592c0861a25b/035fadad-9eba-4726-a427-88058f0933c7"
-					(reference "#PWR078")
+					(reference "#PWR088")
 					(unit 1)
 				)
@@
 		(dnp no)
 		(fields_autoplaced yes)
-		(property "Reference" "#PWR082"
+		(property "Reference" "#PWR092"
 			(at 254 66.04 0)
 			(effects
@@
 			(project "main"
 				(path "/1f57b86c-11e7-4ea8-8f36-592c0861a25b/035fadad-9eba-4726-a427-88058f0933c7"
-					(reference "#PWR082")
+					(reference "#PWR092")
 					(unit 1)
 				)
@@
 		(dnp no)
 		(fields_autoplaced yes)
-		(property "Reference" "#PWR077"
+		(property "Reference" "#PWR087"
 			(at 142.24 85.09 0)
 			(effects
@@
 			(project "main"
 				(path "/1f57b86c-11e7-4ea8-8f36-592c0861a25b/035fadad-9eba-4726-a427-88058f0933c7"
-					(reference "#PWR077")
+					(reference "#PWR087")
 					(unit 1)
 				)
@@
 		(on_board yes)
 		(dnp no)
-		(property "Reference" "#PWR081"
+		(property "Reference" "#PWR091"
 			(at 248.92 68.58 0)
 			(effects
@@
 			(project "main"
 				(path "/1f57b86c-11e7-4ea8-8f36-592c0861a25b/035fadad-9eba-4726-a427-88058f0933c7"
-					(reference "#PWR081")
+					(reference "#PWR091")
 					(unit 1)
 				)
@@
 		(dnp no)
 		(fields_autoplaced yes)
-		(property "Reference" "#PWR069"
+		(property "Reference" "#PWR079"
 			(at 44.45 130.81 0)
 			(effects
@@
 			(project "main"
 				(path "/1f57b86c-11e7-4ea8-8f36-592c0861a25b/035fadad-9eba-4726-a427-88058f0933c7"
-					(reference "#PWR069")
+					(reference "#PWR079")
 					(unit 1)
 				)
@@
 		(dnp no)
 		(fields_autoplaced yes)
-		(property "Reference" "#PWR076"
+		(property "Reference" "#PWR086"
 			(at 129.54 109.22 0)
 			(effects
@@
 			(project "main"
 				(path "/1f57b86c-11e7-4ea8-8f36-592c0861a25b/035fadad-9eba-4726-a427-88058f0933c7"
-					(reference "#PWR076")
+					(reference "#PWR086")
 					(unit 1)
 				)
@@
 		(dnp no)
 		(fields_autoplaced yes)
-		(property "Reference" "#PWR074"
+		(property "Reference" "#PWR084"
 			(at 95.25 60.96 0)
 			(effects
@@
 			(project "main"
 				(path "/1f57b86c-11e7-4ea8-8f36-592c0861a25b/035fadad-9eba-4726-a427-88058f0933c7"
-					(reference "#PWR074")
+					(reference "#PWR084")
 					(unit 1)
 				)
@@
 		(dnp no)
 		(fields_autoplaced yes)
-		(property "Reference" "#PWR080"
+		(property "Reference" "#PWR090"
 			(at 248.92 35.56 0)
 			(effects
@@
 			(project "main"
 				(path "/1f57b86c-11e7-4ea8-8f36-592c0861a25b/035fadad-9eba-4726-a427-88058f0933c7"
-					(reference "#PWR080")
+					(reference "#PWR090")
 					(unit 1)
 				)
@@
 		(dnp no)
 		(fields_autoplaced yes)
-		(property "Reference" "#PWR083"
+		(property "Reference" "#PWR093"
 			(at 262.89 66.04 0)
 			(effects
@@
 			(project "main"
 				(path "/1f57b86c-11e7-4ea8-8f36-592c0861a25b/035fadad-9eba-4726-a427-88058f0933c7"
-					(reference "#PWR083")
+					(reference "#PWR093")
 					(unit 1)
 				)
@@
 		(dnp no)
 		(fields_autoplaced yes)
-		(property "Reference" "#PWR070"
+		(property "Reference" "#PWR080"
 			(at 46.99 63.5 0)
 			(effects
@@
 			(project "RP2350Adev"
 				(path "/1f57b86c-11e7-4ea8-8f36-592c0861a25b/035fadad-9eba-4726-a427-88058f0933c7"
-					(reference "#PWR070")
+					(reference "#PWR080")
 					(unit 1)
 				)
@@
 		(dnp no)
 		(fields_autoplaced yes)
-		(property "Reference" "#PWR073"
+		(property "Reference" "#PWR083"
 			(at 59.69 73.66 0)
 			(effects
@@
 			(project "RP2350Adev"
 				(path "/1f57b86c-11e7-4ea8-8f36-592c0861a25b/035fadad-9eba-4726-a427-88058f0933c7"
-					(reference "#PWR073")
+					(reference "#PWR083")
 					(unit 1)
 				)
@@
 		(dnp no)
 		(fields_autoplaced yes)
-		(property "Reference" "#PWR071"
+		(property "Reference" "#PWR081"
 			(at 46.99 96.52 0)
 			(effects
@@
 			(project "RP2350Adev"
 				(path "/1f57b86c-11e7-4ea8-8f36-592c0861a25b/035fadad-9eba-4726-a427-88058f0933c7"
-					(reference "#PWR071")
+					(reference "#PWR081")
 					(unit 1)
 				)
@@
 		(dnp no)
 		(fields_autoplaced yes)
-		(property "Reference" "#PWR072"
+		(property "Reference" "#PWR082"
 			(at 59.69 40.64 0)
 			(effects
@@
 			(project "main"
 				(path "/1f57b86c-11e7-4ea8-8f36-592c0861a25b/035fadad-9eba-4726-a427-88058f0933c7"
-					(reference "#PWR072")
+					(reference "#PWR082")
 					(unit 1)
 				)
@@
 		(dnp no)
 		(fields_autoplaced yes)
-		(property "Reference" "#PWR079"
+		(property "Reference" "#PWR089"
 			(at 226.06 78.74 0)
 			(effects
@@
 			(project "main"
 				(path "/1f57b86c-11e7-4ea8-8f36-592c0861a25b/035fadad-9eba-4726-a427-88058f0933c7"
-					(reference "#PWR079")
+					(reference "#PWR089")
 					(unit 1)
 				)
@@
 		(lib_id "Switch:SW_DIP_x06")
 		(at 115.57 113.03 0)
-		(unit 1)
-		(exclude_from_sim no)
-		(in_bom yes)
-		(on_board yes)
-		(dnp no)
-		(fields_autoplaced yes)
+		(mirror y)
+		(unit 1)
+		(exclude_from_sim no)
+		(in_bom yes)
+		(on_board yes)
+		(dnp no)
 		(property "Reference" "SW1"
 			(at 115.57 97.79 0)
